File: analog-toolkit.kicad_pcb (KiCad board)
At the start: 2 copper layers, 50 x 36 mm, 55 parts, among them J1 USB_C, J2 IO, J3 UART, J4 I2C, J5 VBUS, J6 3.3V, J7 OPAMP, J8 ADC, P1 TC2030, Q1 AO3400A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

Commit message: updated version
Parts:
- turned J5 to -175 degrees
Other:
- board text added: "STM32G4 Analog toolkit Jana Marie 2025"
- board text removed: "STM32G4 Analog toolkit Jana Marie 2023"

Commit message: bumped improved version
Parts:
- C10, C11, C12, C13, C8, C9: value 100n -> 10n
- U3: value STM32G431xB -> STM32G431KBT6
- turned D1 to 180 degrees
Connections:
- D1 pad 1: LED1 -> Net-(D1-RK)
- D1 pad 2: Net-(D1-Pad2) -> LED1
- D1 pad 3: Net-(D1-Pad3) -> Net-(D1-BK)
- D1 pad 4: Net-(D1-Pad4) -> LED1
- D1 pad 5: LED1 -> Net-(D1-GA)
- D1 pad 6: Net-(D1-Pad6) -> Net-(D1-RA)
- Q1 pad 3: Net-(D1-Pad3) -> Net-(D1-RA)
- R2 pad 2: Net-(D1-Pad6) -> Net-(D1-BK)
- R3 pad 1: Net-(D1-Pad2) -> Net-(D1-GA)
- R4 pad 2: Net-(D1-Pad4) -> Net-(D1-RK)
Routing:
- net Net-(D1-Pad6): track 7.09 -> 0.00 mm
- net Net-(D1-BK): track 0.00 -> 7.09 mm
- net Net-(D1-RA): track 0.00 -> 3.06 mm
- net Net-(D1-Pad3): track 3.06 -> 0.00 mm
- net Net-(D1-Pad2): track 2.50 -> 0.00 mm
- net Net-(D1-GA): track 0.00 -> 2.50 mm
- net Net-(D1-RK): track 0.00 -> 2.05 mm
- net Net-(D1-Pad4): track 2.05 -> 0.00 mm
