File: analog-toolkit.kicad_pcb (KiCad board)
At the start: 2 copper layers, 50 x 36 mm, 55 parts, among them J1 USB_C, J2 IO, J3 UART, J4 I2C, J5 VBUS, J6 3.3V, J7 OPAMP, J8 ADC, P1 TC2030, Q1 AO3400A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

Commit message: updated boards, replaced RGB led
Parts:
- removed Q1: AO3400A, Package_TO_SOT_SMD:SOT-23
- removed R4: 5k1, otter:R_0402
- added D2: ACT, LED_SMD:LED_0805_2012Metric, F.Cu at (138.5, 134.0)
- D1: value LED_RGB -> PWR; footprint LED_SMD:LED_RGB_5050-6 -> LED_SMD:LED_0805_2012Metric
- R2, R3: value 5k1 -> 22k
- moved D1 5.59 mm to (138.5, 131.0)
- moved R2 4.83 mm to (141.0, 134.0), turned to -90 degrees
- moved R3 1.82 mm to (141.0, 131.0), turned to -90 degrees
Connections:
- D1 pad 1: Net-(D1-RK) -> Net-(D1-K)
- D1 pad 2: LED1 -> LED2
- R2 pad 1: LED2 -> Net-(D2-K)
- R2 pad 2: Net-(D1-BK) -> GND
- R3 pad 1: Net-(D1-GA) -> GND
- R3 pad 2: LED2 -> Net-(D1-K)
Routing:
- net LED1: track 44.3 -> 27.8 mm
- net Net-(D1-BK): track 7.09 -> 0.00 mm
- net LED2: track 28.8 -> 25.7 mm
- net Net-(D1-RA): track 3.06 -> 0.00 mm
- net Net-(D1-GA): track 2.50 -> 0.00 mm
- net Net-(D1-RK): track 2.05 -> 0.00 mm
- net Net-(D2-K): track 0.00 -> 1.76 mm
- net Net-(D1-K): track 0.00 -> 1.76 mm
- net GND: vias 152 -> 143
Other:
- board text added: "ACT"
- board text added: "PWR"
- board text added: "STM32G4 Analog toolkit Jana Marie 2026"
- board text removed: "STM32G4 Analog toolkit Jana Marie 2025"

Commit message: updated board with jlc-specific parts
Parts:
- SW1: footprint Button_Switch_SMD:SW_SPST_PTS810 -> Button_Switch_SMD:SW_SPST_TS-1088-xR020
- U1: value AP2204R-3.3 -> AP2204RA-3.3
- moved R1 7.11 mm to (122.6, 104.5)
- moved G*** 0.45 mm to (128.4, 103.7)
- turned C1 to -90 degrees
Connections:
- U1 pad 1: VBUS -> GND
- U1 pad 2: GND -> VBUS
Routing:
- net Net-(U3-PB8-BOOT0): track 17.1 -> 13.9 mm
- net VBUS: track 16.9 -> 18.0 mm
- net +3V3: track 85.5 -> 86.0 mm
- net GND: vias 143 -> 147
